File: schematics/hail-met-v0/hail-met-v0.sch (EAGLE design)
At the start: 87 parts, among them IC1 MCP73871, U1 ATMEGA328P, U2 TLC5917ID, Y1 16MHZ

Commit message: updated schematic with pins (CPU pins not verified)
Connections:
- net N$30 renamed CHG_STAT
- net N$38 renamed BT_CONN
- net N$40 renamed BT_PAIR
- removed net BTH_CMD: U$3.GPIO9, U1.PD3(INT1)
- removed net BTH_EVENT: U$3.GPIO2, U1.PD2(INT0)
- removed net N$14: U2.LE(ED1)
- removed net N$28: U1.PC1(ADC1)
- removed net N$29: U1.PC2(ADC2)
- removed net N$39: U1.PD6(AIN0)
- removed net N$41: U1.PB0(ICP)
- removed net N$42: U1.PB2(SS/OC1B)
- removed net N$44: U1.PB4(MISO)
- new net BT_CMD: U$3.GPIO9, U1.PB2(SS/OC1B)
- new net BT_DISC: U1.PD4(XCK/T0)
- new net BT_EVENT: U$3.GPIO2, U1.PB0(ICP)
- new net LED_LE: U1.PB4(MISO), U2.LE(ED1)
- new net SIG_LEFT: U1.PD2(INT0)
- new net SIG_RIGHT: U1.PD3(INT1)
- net CHG_DONE: now also U1.PC2(ADC2)
- net CHG_PWR: now also U1.PC1(ADC1)
- net DEV_EN: now also U1.PB1(OC1A); no longer U1.PD4(XCK/T0)
- net GND: now also ATM_PWR.4
- net LED_OE: now also U1.PD6(AIN0); no longer U1.PB1(OC1A)
- net N$32: no longer ATM_PWR.4
Other:
- note added: "Note: Processor pins do not match button pins yet, and pins and there is 1 less pin than expected. ADC6/ ADC7 were factored in as pins, but not on standard Arduino IDE(?)"
Changed lines of the file:
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@@
 <part name="C1" library="SparkFun-Passives" deviceset="CAP" device="0805" value="0.1uF"/>
 <part name="R1" library="SparkFun-Passives" deviceset="RESISTOR" device="0805-RES"/>
-<part name="GND17" library="SparkFun" deviceset="GND" device=""/>
 <part name="R2" library="SparkFun-Passives" deviceset="RESISTOR" device="0805-RES"/>
 <part name="R10" library="SparkFun-Passives" deviceset="RESISTOR" device="0805-RES"/>
@@
 <text x="71.12" y="-78.74" size="1.778" layer="91" align="bottom-right">Design:
 Validate:</text>
-<text x="243.84" y="-50.8" size="1.778" layer="91">Names:
+<text x="238.76" y="-50.8" size="1.778" layer="91">Names:
 ------
 LED0-LF  Left Front
@@
 LM317DCYR
 296-12602-1-ND</text>
+<text x="109.22" y="10.16" size="1.778" layer="94">Note: Processor pins do not match
+button pins yet, and pins and there
+is 1 less pin than expected. ADC6/
+ADC7 were factored in as pins, but
+not on standard Arduino IDE(?)</text>
 </plain>
 <instances>
@@
 <instance part="C1" gate="G$1" x="73.66" y="91.44" rot="R180"/>
 <instance part="R1" gate="G$1" x="129.54" y="-55.88" rot="R180"/>
-<instance part="GND17" gate="1" x="124.46" y="-58.42"/>
 <instance part="R2" gate="G$1" x="193.04" y="-33.02" rot="R180"/>
 <instance part="R10" gate="G$1" x="193.04" y="-48.26" rot="R180"/>
@@
 </segment>
 <segment>
-<pinref part="R1" gate="G$1" pin="2"/>
-<pinref part="GND17" gate="1" pin="GND"/>
-</segment>
-<segment>
 <pinref part="GND18" gate="1" pin="GND"/>
 <pinref part="U$3" gate="G$1" pin="GND0"/>
@@
 <pinref part="R12" gate="G$1" pin="2"/>
 </segment>
+<segment>
+<pinref part="ATM_PWR" gate="G$1" pin="4"/>
+<wire x1="60.96" y1="-25.4" x2="73.66" y2="-25.4" width="0.1524" layer="91"/>
+<label x="60.96" y="-25.4" size="1.778" layer="95"/>
+</segment>
+<segment>
+<pinref part="R1" gate="G$1" pin="2"/>
+<wire x1="119.38" y1="-55.88" x2="124.46" y2="-55.88" width="0.1524" layer="91"/>
+<label x="119.38" y="-55.88" size="1.778" layer="95"/>
+</segment>
 </net>
 <net name="VIN" class="0">
@@
 <segment>
 <pinref part="U2" gate="A" pin="~OE(ED2)"/>
-<wire x1="134.62" y1="-63.5" x2="121.92" y2="-63.5" width="0.1524" layer="91"/>
-<label x="121.92" y="-63.5" size="1.778" layer="95"/>
-</segment>
-<segment>
-<pinref part="U1" gate="G$1" pin="PB1(OC1A)"/>
-<wire x1="132.08" y1="38.1" x2="142.24" y2="38.1" width="0.1524" layer="91"/>
-<label x="134.62" y="38.1" size="1.778" layer="95"/>
-</segment>
-</net>
-<net name="N$14" class="0">
+<wire x1="134.62" y1="-63.5" x2="119.38" y2="-63.5" width="0.1524" layer="91"/>
+<label x="119.38" y="-63.5" size="1.778" layer="95"/>
+</segment>
+<segment>
+<pinref part="U1" gate="G$1" pin="PD6(AIN0)"/>
+<wire x1="132.08" y1="48.26" x2="142.24" y2="48.26" width="0.1524" layer="91"/>
+<label x="134.62" y="48.26" size="1.778" layer="95"/>
+</segment>
+</net>
+<net name="LED_LE" class="0">
 <segment>
 <pinref part="U2" gate="A" pin="LE(ED1)"/>
-<wire x1="134.62" y1="-60.96" x2="121.92" y2="-60.96" width="0.1524" layer="91"/>
+<wire x1="134.62" y1="-60.96" x2="119.38" y2="-60.96" width="0.1524" layer="91"/>
+<label x="119.38" y="-60.96" size="1.778" layer="95"/>
+</segment>
+<segment>
+<pinref part="U1" gate="G$1" pin="PB4(MISO)"/>
+<wire x1="132.08" y1="30.48" x2="142.24" y2="30.48" width="0.1524" layer="91"/>
+<label x="134.62" y="30.48" size="1.778" layer="95"/>
 </segment>
 </net>
@@
 <segment>
 <pinref part="U2" gate="A" pin="CLK"/>
-<wire x1="134.62" y1="-53.34" x2="121.92" y2="-53.34" width="0.1524" layer="91"/>
-<label x="121.92" y="-53.34" size="1.778" layer="95"/>
+<wire x1="134.62" y1="-53.34" x2="119.38" y2="-53.34" width="0.1524" layer="91"/>
+<label x="119.38" y="-53.34" size="1.778" layer="95"/>
 </segment>
 <segment>
@@
 <pinref part="R26" gate="G$1" pin="2"/>
 </segment>
+<segment>
+<pinref part="U1" gate="G$1" pin="PC1(ADC1)"/>
+<wire x1="132.08" y1="83.82" x2="142.24" y2="83.82" width="0.1524" layer="91"/>
+<label x="134.62" y="83.82" size="1.778" layer="95"/>
+</segment>
 </net>
 <net name="CHG_DONE" class="0">
@@
 <pinref part="R25" gate="G$1" pin="2"/>
 <wire x1="-175.26" y1="43.18" x2="-139.7" y2="43.18" width="0.1524" layer="91"/>
+</segment>
+<segment>
+<pinref part="U1" gate="G$1" pin="PC2(ADC2)"/>
+<wire x1="132.08" y1="81.28" x2="142.24" y2="81.28" width="0.1524" layer="91"/>
+<label x="134.62" y="81.28" size="1.778" layer="95"/>
 </segment>
 </net>
@@
 </segment>
 </net>
-<net name="N$28" class="0">
-<segment>
-<pinref part="U1" gate="G$1" pin="PC1(ADC1)"/>
-<wire x1="132.08" y1="83.82" x2="142.24" y2="83.82" width="0.1524" layer="91"/>
-</segment>
-</net>
-<net name="N$29" class="0">
-<segment>
-<pinref part="U1" gate="G$1" pin="PC2(ADC2)"/>
-<wire x1="132.08" y1="81.28" x2="142.24" y2="81.28" width="0.1524" layer="91"/>
-</segment>
-</net>
-<net name="N$30" class="0">
+<net name="CHG_STAT" class="0">
 <segment>
 <pinref part="U1" gate="G$1" pin="PC3(ADC3)"/>
 <wire x1="132.08" y1="78.74" x2="142.24" y2="78.74" width="0.1524" layer="91"/>
+<label x="134.62" y="78.74" size="1.778" layer="95"/>
 </segment>
 </net>
@@
 <pinref part="U1" gate="G$1" pin="ADC6"/>
 <wire x1="132.08" y1="71.12" x2="142.24" y2="71.12" width="0.1524" layer="91"/>
+<label x="134.62" y="71.12" size="1.778" layer="95"/>
 </segment>
 </net>
@@
 <pinref part="U1" gate="G$1" pin="ADC7"/>
 <wire x1="132.08" y1="68.58" x2="142.24" y2="68.58" width="0.1524" layer="91"/>
-</segment>
-</net>
-<net name="N$38" class="0">
+<label x="134.62" y="68.58" size="1.778" layer="95"/>
+</segment>
+</net>
+<net name="BT_CONN" class="0">
 <segment>
 <pinref part="U1" gate="G$1" pin="PD5(T1)"/>
 <wire x1="132.08" y1="50.8" x2="142.24" y2="50.8" width="0.1524" layer="91"/>
-</segment>
-</net>
-<net name="N$39" class="0">
-<segment>
-<pinref part="U1" gate="G$1" pin="PD6(AIN0)"/>
-<wire x1="132.08" y1="48.26" x2="142.24" y2="48.26" width="0.1524" layer="91"/>
-</segment>
-</net>
-<net name="N$40" class="0">
+<label x="134.62" y="50.8" size="1.778" layer="95"/>
+</segment>
+</net>
+<net name="BT_PAIR" class="0">
 <segment>
 <pinref part="U1" gate="G$1" pin="PD7(AIN1)"/>
 <wire x1="132.08" y1="45.72" x2="142.24" y2="45.72" width="0.1524" layer="91"/>
-</segment>
-</net>
-<net name="N$41" class="0">
+<label x="134.62" y="45.72" size="1.778" layer="95"/>
+</segment>
+</net>
+<net name="BT_EVENT" class="0">
 <segment>
 <pinref part="U1" gate="G$1" pin="PB0(ICP)"/>
 <wire x1="132.08" y1="40.64" x2="142.24" y2="40.64" width="0.1524" layer="91"/>
-</segment>
-</net>
-<net name="N$42" class="0">
+<label x="134.62" y="40.64" size="1.778" layer="95"/>
+</segment>
+<segment>
+<pinref part="U$3" gate="G$1" pin="GPIO2"/>
+<wire x1="-149.86" y1="-40.64" x2="-170.18" y2="-40.64" width="0.1524" layer="91"/>
+<label x="-170.18" y="-40.64" size="1.778" layer="95"/>
+</segment>
+</net>
+<net name="BT_CMD" class="0">
 <segment>
 <pinref part="U1" gate="G$1" pin="PB2(SS/OC1B)"/>
 <wire x1="132.08" y1="35.56" x2="142.24" y2="35.56" width="0.1524" layer="91"/>
+<label x="134.62" y="35.56" size="1.778" layer="95"/>
+</segment>
+<segment>
+<pinref part="U$3" gate="G$1" pin="GPIO9"/>
+<wire x1="-149.86" y1="-55.88" x2="-170.18" y2="-55.88" width="0.1524" layer="91"/>
+<label x="-170.18" y="-55.88" size="1.778" layer="95"/>
 </segment>
 </net>
@@
 <segment>
 <pinref part="U2" gate="A" pin="SDI"/>
-<wire x1="134.62" y1="-50.8" x2="121.92" y2="-50.8" width="0.1524" layer="91"/>
-<label x="121.92" y="-50.8" size="1.778" layer="95"/>
-</segment>
-</net>
-<net name="N$44" class="0">
-<segment>
-<pinref part="U1" gate="G$1" pin="PB4(MISO)"/>
-<wire x1="132.08" y1="30.48" x2="142.24" y2="30.48" width="0.1524" layer="91"/>
+<wire x1="134.62" y1="-50.8" x2="119.38" y2="-50.8" width="0.1524" layer="91"/>
+<label x="119.38" y="-50.8" size="1.778" layer="95"/>
 </segment>
 </net>
@@
 <net name="N$32" class="0">
 <segment>
-<pinref part="ATM_PWR" gate="G$1" pin="4"/>
-<wire x1="60.96" y1="-25.4" x2="73.66" y2="-25.4" width="0.1524" layer="91"/>
-<label x="60.96" y="-25.4" size="1.778" layer="95"/>
-</segment>
-<segment>
 <pinref part="ATM_PC" gate="G$1" pin="4"/>
 <wire x1="86.36" y1="-25.4" x2="99.06" y2="-25.4" width="0.1524" layer="91"/>
@@
 </segment>
 </net>
-<net name="BTH_EVENT" class="0">
-<segment>
-<pinref part="U$3" gate="G$1" pin="GPIO2"/>
-<wire x1="-149.86" y1="-40.64" x2="-170.18" y2="-40.64" width="0.1524" layer="91"/>
-<label x="-170.18" y="-40.64" size="1.778" layer="95"/>
-</segment>
-<segment>
-<pinref part="U1" gate="G$1" pin="PD2(INT0)"/>
-<wire x1="132.08" y1="58.42" x2="142.24" y2="58.42" width="0.1524" layer="91"/>
-<label x="134.62" y="58.42" size="1.778" layer="95"/>
-</segment>
-</net>
-<net name="BTH_CMD" class="0">
-<segment>
-<pinref part="U$3" gate="G$1" pin="GPIO9"/>
-<wire x1="-149.86" y1="-55.88" x2="-170.18" y2="-55.88" width="0.1524" layer="91"/>
-<label x="-170.18" y="-55.88" size="1.778" layer="95"/>
-</segment>
-<segment>
-<pinref part="U1" gate="G$1" pin="PD3(INT1)"/>
-<wire x1="132.08" y1="55.88" x2="142.24" y2="55.88" width="0.1524" layer="91"/>
-<label x="134.62" y="55.88" size="1.778" layer="95"/>
-</segment>
-</net>
 <net name="MPU_INT" class="0">
 <segment>
@@
 </segment>
 <segment>
+<pinref part="U1" gate="G$1" pin="PB1(OC1A)"/>
+<wire x1="132.08" y1="38.1" x2="142.24" y2="38.1" width="0.1524" layer="91"/>
+<label x="134.62" y="38.1" size="1.778" layer="95"/>
+</segment>
+</net>
+<net name="SIG_LEFT" class="0">
+<segment>
+<pinref part="U1" gate="G$1" pin="PD2(INT0)"/>
+<wire x1="132.08" y1="58.42" x2="142.24" y2="58.42" width="0.1524" layer="91"/>
+<label x="134.62" y="58.42" size="1.778" layer="95"/>
+</segment>
+</net>
+<net name="SIG_RIGHT" class="0">
+<segment>
+<pinref part="U1" gate="G$1" pin="PD3(INT1)"/>
+<wire x1="132.08" y1="55.88" x2="142.24" y2="55.88" width="0.1524" layer="91"/>
+<label x="134.62" y="55.88" size="1.778" layer="95"/>
+</segment>
+</net>
+<net name="BT_DISC" class="0">
+<segment>
 <pinref part="U1" gate="G$1" pin="PD4(XCK/T0)"/>

Commit message: modified schematic slightly and began board layout.
Parts:
- removed R15, R25, R26: 1K, SparkFun-Passives:RESISTOR0805-RES
- added J1: AVR_SPI_PRG_6PTH, SparkFun-Connectors:AVR_SPI_PRG_6PTH
Connections:
- new net N$21: J1.2
- net 3.3V: no longer R13.2, R15.1, R25.1, R26.1, R5.2, R6.2
- net CHG_DONE: no longer R25.2
- net CHG_PWR: no longer R26.2
- net CHG_STAT1: no longer R15.2
- net CHG_VOUT: now also C7.1, U$1.IN
- net GND: now also J1.6
- net LED_CLK: now also J1.3
- net LED_LE: now also J1.1
- net LED_SDI: now also J1.4
- net RESET: now also J1.5
- net VCHG: now also R13.2, R5.2, R6.2
- net VIN: no longer C7.1, U$1.IN
Other:
- note added: "RT1 = 1k, RT2 = 150k"
- note removed: "RT1 = TBD, RT2 = TBD"

Commit message: updated schematic/board and datasheets
Parts:
- removed JP_BATT, JP_SOLAR: (no value), adafruit:JST_2PIN-SMT-RA
- removed MIC: M02PTH, SparkFun-Connectors:M02PTH
- added JBATT, JSOLAR, MIC_L, MIC_R: (no value), adafruit:JST_2PIN-SMT
- added Q1: (no value), semicon-smd-ipc:NPN-TRANSISTOR_SOT89
- R12: value (none) -> 10k
- SPK_L, SPK_R: value M02PTH -> (none); device SparkFun-Connectors:M02PTH -> adafruit:JST_2PIN-SMT
- renumbered LED7-LB to LED7-FREE, U$4 to LM4871, U2 to TLC5917ID
Connections:
- net CHG_STAT renamed C
- removed net N$33: U1.ADC6
- removed net N$69: U$3.UART_TX
- removed net N$70: U$3.UART_RX
- removed net SIG_LEFT: U1.PD2(INT0)
- removed net SIG_RIGHT: U1.PD3(INT1)
- new net A: U1.PC1(ADC1)
- new net B: U1.PC2(ADC2)
- new net BT_GPIO10: JP4.8, U$3.GPIO10
- new net BT_GPIO2: JP4.1
- new net BT_GPIO3: JP4.2, U$3.GPIO3
- new net BT_GPIO4: JP4.3, U$3.GPIO4
- new net BT_GPIO5: JP4.4, U$3.GPIO5
- new net BT_GPIO6: JP4.5, U$3.GPIO6
- new net BT_GPIO7: JP4.6, U$3.GPIO7
- new net BT_GPIO9: JP4.7
- new net LED_CREE: Q1.B, U1.PC0(ADC0)
- new net N$19: Q1.C, R24.2
- net 3.3V: now also U$3.VDD; no longer LED_CREE.1
- net AMB_IN: now also U1.ADC6; no longer U1.PC0(ADC0)
- net CHG_DONE: no longer U1.PC2(ADC2)
- net CHG_PWR: no longer U1.PC1(ADC1)
- net GND: now also JBATT.2, JSOLAR.2, LM4871.SHUTDWN, Q1.E; no longer JP_BATT.2, JP_SOLAR.2
- net MIC_L+: now also MIC_L.1, U$3.MIC_L+; no longer JP4.8
- net MIC_L-: now also MIC_L.2, U$3.MIC_L-; no longer JP4.6
- net MIC_R+: now also MIC_R.1, U$3.MIC_R+; no longer JP4.7
- net MIC_R-: now also MIC_R.2, U$3.MIC_R-; no longer JP4.5
- net N$80: now also JSOLAR.1; no longer JP_SOLAR.1
- net RXD: now also U$3.UART_TX
- net SPKR_L+: no longer JP4.1
- net SPKR_L-: no longer JP4.3
- net SPKR_R+: no longer JP4.2
- net SPKR_R-: no longer JP4.4
- net SW_TL: now also U1.PD2(INT0)
- net SW_TR: now also U1.PD3(INT1)
- net TXD: now also U$3.UART_RX
- net VBATT: now also JBATT.1; no longer JP_BATT.1
- net VCHG: now also LED_CREE.1
Other:
- note added: "Do we need these jumpers?"
- note added: "Mic required to have dBV between -40 and -60"
- note added: "Names: ------ LED0-LF Left Front LED0-IL Indicator Left LED1-LM Left Middle LED2-LR Left Rear LED3-HR Headlight Front LED4-RF Right Front LED4-IR Indicator Right LED5-RM Right Middle LED6-RR Right Rear LED7-FREE"
- note removed: "Names: ------ LED0-LF Left Front LED0-IL Indicator Left LED1-LM Left Middle LED2-LR Left Rear LED3-HR Headlight Front LED4-RF Right Front LED4-IR Indicator Right LED5-RM Right Middle LED6-RR Right Rear LED7-LB Low-battery indicator"
- note removed: "Step-up converter for USB phone port"
- moved on the sheet: R12, SPK_L, SPK_R, U$5
