File: schematics/hail-met-v1/hail-met-v1.brd (EAGLE design)
At the start: 77.1 x 61 mm, 99 parts, among them IC1 MCP73871, J1 AVR_SPI_PRG_6PTH, U1 ATMEGA328P, Y1 16MHZ

Commit message: updated schematics (v0, v1) and datasheets
Parts:
- removed R8: 240, SparkFun-Passives:0805
- removed R9: 390, SparkFun-Passives:0805
- removed U$1: V_REG_317SMD, SparkFun:SOT223
- added IC2: 78L05Z, adafruit:TO92
- C7: value 10uF -> 0.1uF
- C8: value 22pF -> 2.2uF
- R11: value 100K -> 8.2K
- R3: value (none) -> 270K
- R4: value (none) -> 100K
- RT1: value (none) -> 0
- RT2: value (none) -> 82K
Connections:
- removed net N$4: R8.1, R9.2, U$1.1
- net 3.3V: now also IC2.1; no longer R8.2, U$1.2
- net GND: now also IC2.2; no longer R9.1
- net VIN: now also IC2.3; no longer U$1.3
Routing:
- net N$4: track 7.50 -> 0.00 mm
- net GND: track 56.4 -> 55.6 mm

Commit message: updated and routed v1 board
Routing:
- net N$27: track 0.00 -> 33.2 mm, vias 0 -> 2
- net N$26: track 0.00 -> 32.5 mm, vias 0 -> 2
- net N$14: track 0.00 -> 30.3 mm, vias 0 -> 2
- net 3.3V: track 8.38 -> 7.49 mm
- net BT_CMD: track 50.2 -> 49.6 mm
Other:
- board text added: "Hail-met v1 Ben Wang, Brian Margosian, Brian Daniels, Alex Jaeckel, Patrick Hayes EECS 473 University of Michigan (C) 2014"
