File: schematics/hail-met-v1/hail-met-v1.brd (EAGLE design)
At the start: 77.1 x 61 mm, 97 parts, among them IC1 MCP73871, IC2 78L05Z, J1 AVR_SPI_PRG_6PTH, U1 ATMEGA328P, Y1 16MHZ

Commit message: updated board v1
Parts:
- removed MIC_R: (no value), adafruit:JST-PH-2-SMT
Connections:
- removed net MIC_R+: MIC_R.1, U$3.MIC_R+
- removed net MIC_R-: MIC_R.2, U$3.MIC_R-
Routing:
- net MIC_R-: track 28.0 -> 0.00 mm
- net MIC_R+: track 26.7 -> 0.00 mm, vias 2 -> 0
- net DEV_EN: track 39.0 -> 40.1 mm
- net GND: track 55.6 -> 56.6 mm
Other:
- outline, holes or cut-outs redrawn
Changed lines of the file:
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@@
 <layer number="27" name="tValues" color="7" fill="1" visible="yes" active="yes"/>
 <layer number="28" name="bValues" color="7" fill="1" visible="yes" active="yes"/>
-<layer number="29" name="tStop" color="7" fill="3" visible="no" active="yes"/>
-<layer number="30" name="bStop" color="7" fill="6" visible="no" active="yes"/>
-<layer number="31" name="tCream" color="7" fill="4" visible="no" active="yes"/>
-<layer number="32" name="bCream" color="7" fill="5" visible="no" active="yes"/>
+<layer number="29" name="tStop" color="7" fill="3" visible="yes" active="yes"/>
+<layer number="30" name="bStop" color="7" fill="6" visible="yes" active="yes"/>
+<layer number="31" name="tCream" color="7" fill="4" visible="yes" active="yes"/>
+<layer number="32" name="bCream" color="7" fill="5" visible="yes" active="yes"/>
 <layer number="33" name="tFinish" color="6" fill="3" visible="no" active="yes"/>
 <layer number="34" name="bFinish" color="6" fill="6" visible="no" active="yes"/>
@@
 <board>
 <plain>
-<wire x1="0" y1="0" x2="77.14" y2="0" width="0" layer="20"/>
-<wire x1="77.14" y1="0" x2="77.14" y2="60.95" width="0" layer="20"/>
-<wire x1="77.14" y1="60.95" x2="0" y2="60.95" width="0" layer="20"/>
-<wire x1="0" y1="60.95" x2="0" y2="0" width="0" layer="20"/>
+<wire x1="0" y1="57.775" x2="0" y2="3.175" width="0" layer="20"/>
+<wire x1="0" y1="3.175" x2="3.175" y2="0" width="0" layer="20" curve="90"/>
+<wire x1="3.175" y1="0" x2="73.965" y2="0" width="0" layer="20"/>
+<wire x1="73.965" y1="0" x2="77.14" y2="3.175" width="0" layer="20" curve="90"/>
+<wire x1="77.14" y1="3.175" x2="77.14" y2="57.775" width="0" layer="20"/>
+<wire x1="77.14" y1="57.775" x2="73.965" y2="60.95" width="0" layer="20" curve="90"/>
+<wire x1="73.965" y1="60.95" x2="3.175" y2="60.95" width="0" layer="20"/>
+<wire x1="3.175" y1="60.95" x2="0" y2="57.775" width="0" layer="20" curve="90"/>
 <dimension x1="0" y1="60.95" x2="77.14" y2="60.95" x3="38.57" y3="68.58" textsize="1.778" layer="19" unit="inch"/>
 <dimension x1="77.14" y1="60.95" x2="77.47" y2="0" x3="100.157453125" y3="30.59873125" textsize="1.778" layer="19" unit="inch"/>
-<text x="67.0814" y="60.4012" size="0.8128" layer="25" rot="R90" align="top-right">VDD
+<text x="64.315340625" y="60.645040625" size="0.8128" layer="25" rot="R90" align="top-right">VDD
 GND
 INT
@@
 <attribute name="VALUE" x="17.78" y="10.16" size="1.27" layer="27" font="vector" rot="R180"/>
 </element>
-<element name="MIC_R" library="adafruit" package="JST-PH-2-SMT" value="" x="6.4008" y="2.5146" smashed="yes" rot="R180">
-<attribute name="NAME" x="11.4554" y="9.8552" size="1.27" layer="25" font="vector" rot="R180"/>
-<attribute name="VALUE" x="8.9408" y="10.1346" size="1.27" layer="27" font="vector" rot="R180"/>
-</element>
 <element name="SPK_L" library="adafruit" package="JST-PH-2-SMT" value="" x="2.54" y="12.7" smashed="yes" rot="R90">
 <attribute name="NAME" x="9.779" y="11.2014" size="1.27" layer="25" font="vector" rot="R90"/>
@@
 <vertex x="42.1386" y="1.5748"/>
 <vertex x="40.5892" y="3.1242"/>
-<vertex x="6.731" y="3.1242"/>
-<vertex x="4.7244" y="6.4008"/>
+<vertex x="9.017" y="3.1242"/>
+<vertex x="4.9784" y="6.9088"/>
 <vertex x="4.7244" y="27.6098"/>
 <vertex x="3.1242" y="27.94"/>
@@
 </polygon>
 <via x="25.4508" y="5.1308" extent="1-16" drill="0.6" shape="octagon"/>
-<via x="31.3436" y="37.9476" extent="1-16" drill="0.6" shape="octagon"/>
-<wire x1="30.353" y1="37.9476" x2="31.3436" y2="37.9476" width="0.4064" layer="1"/>
+<via x="32.3596" y="37.9476" extent="1-16" drill="0.6" shape="octagon"/>
+<wire x1="30.353" y1="37.9476" x2="32.3596" y2="37.9476" width="0.4064" layer="1"/>
 <contactref element="JBATT" pad="2"/>
 <contactref element="JSOLAR" pad="1"/>
@@
 <vertex x="30.226" y="36.0426"/>
 <vertex x="30.226" y="35.3314"/>
-<vertex x="31.3944" y="34.163"/>
 <vertex x="35.5092" y="30.0482"/>
 <vertex x="35.5092" y="25.8318"/>
 <vertex x="36.9316" y="24.4094"/>
-<vertex x="36.9316" y="17.8816"/>
 <vertex x="36.9316" y="16.2814"/>
 <vertex x="37.8968" y="15.3162"/>
 <vertex x="38.5318" y="15.3162"/>
 <vertex x="39.2938" y="16.0782"/>
-<vertex x="39.2938" y="26.9748"/>
-<vertex x="41.1226" y="28.8036"/>
+<vertex x="39.2938" y="26.2128"/>
+<vertex x="41.1226" y="28.0416"/>
 <vertex x="42.5704" y="28.8036"/>
 <vertex x="43.7896" y="30.0228"/>
@@
 <wire x1="20.5884" y1="56.7038" x2="21.4376" y2="55.8546" width="0.6096" layer="1"/>
 </signal>
-<signal name="MIC_R-">
-<contactref element="U$3" pad="MIC_R-"/>
-<contactref element="MIC_R" pad="2"/>
-<wire x1="5.4008" y1="4.3146" x2="5.4008" y2="7.1026" width="0.3048" layer="1"/>
-<wire x1="5.4008" y1="7.1026" x2="7.3914" y2="9.0932" width="0.3048" layer="1"/>
-<wire x1="7.3914" y1="9.0932" x2="16.637" y2="9.0932" width="0.3048" layer="1"/>
-<wire x1="16.637" y1="9.0932" x2="17.653" y2="8.0772" width="0.3048" layer="1"/>
-<wire x1="17.653" y1="8.0772" x2="29.2782" y2="8.0772" width="0.3048" layer="1"/>
-<wire x1="29.2782" y1="8.0772" x2="29.3244" y2="8.1234" width="0.3048" layer="1"/>
-</signal>
 <signal name="MIC_L-">
 <contactref element="U$3" pad="MIC_L-"/>
@@
 <wire x1="19.1278" y1="9.3234" x2="29.3244" y2="9.3234" width="0.3048" layer="1"/>
 </signal>
-<signal name="MIC_R+">
-<contactref element="U$3" pad="MIC_R+"/>
-<contactref element="MIC_R" pad="1"/>
-<wire x1="7.4008" y1="4.3146" x2="7.4008" y2="6.08" width="0.3048" layer="1"/>
-<wire x1="7.4008" y1="6.08" x2="9.5504" y2="8.2296" width="0.3048" layer="1"/>
-<via x="9.5504" y="8.2296" extent="1-16" drill="0.3556"/>
-<wire x1="9.5504" y1="8.2296" x2="9.5504" y2="10.3124" width="0.3048" layer="16"/>
-<via x="9.5504" y="10.3124" extent="1-16" drill="0.3556"/>
-<wire x1="9.5504" y1="10.3124" x2="29.1134" y2="10.3124" width="0.3048" layer="1"/>
-<wire x1="29.1134" y1="10.3124" x2="29.3244" y2="10.5234" width="0.3048" layer="1"/>
-</signal>
 <signal name="MPU_INT">
 <contactref element="MPU-6050" pad="3"/>
@@
 <wire x1="28.321" y1="25.0444" x2="27.3812" y2="25.9842" width="0.2032" layer="1"/>
 <via x="27.3812" y="25.9842" extent="1-16" drill="0.4064"/>
-<wire x1="24.4348" y1="34.5948" x2="24.4348" y2="36.7538" width="0.254" layer="16"/>
-<via x="24.4348" y="36.7538" extent="1-16" drill="0.4064"/>
-<wire x1="24.4348" y1="36.7538" x2="22.5552" y2="36.7538" width="0.254" layer="1"/>
+<wire x1="24.4348" y1="34.5948" x2="24.4348" y2="37.5158" width="0.254" layer="16"/>
+<via x="24.4348" y="37.5158" extent="1-16" drill="0.4064"/>
 <wire x1="22.5552" y1="36.7538" x2="21.19" y2="38.119" width="0.254" layer="1"/>
 <wire x1="21.19" y1="38.119" x2="21.19" y2="39.8526" width="0.254" layer="1"/>
@@
 <wire x1="30.5308" y1="34.4424" x2="24.5872" y2="34.4424" width="0.254" layer="16"/>
 <wire x1="24.5872" y1="34.4424" x2="24.4348" y2="34.5948" width="0.254" layer="16"/>
+<wire x1="22.5552" y1="36.7538" x2="23.6728" y2="36.7538" width="0.254" layer="1"/>
+<wire x1="23.6728" y1="36.7538" x2="24.4348" y2="37.5158" width="0.254" layer="1"/>
 </signal>
 <signal name="MPU_VIO">

Commit message: modified board with audio amp values
Connections:
- removed net PC1: AT_PINS.7, U1.24
- net CHG_LOWBATT: now also AT_PINS.7, U1.24
Routing:
- net CHG_LOWBATT: track 10.2 -> 17.5 mm, vias 1 -> 2
- net PC1: track 7.30 -> 0.00 mm, vias 1 -> 0
Changed lines of the file:
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@@
 <wire x1="52.1564" y1="21.783" x2="52.1564" y2="19.5166" width="0.4064" layer="1"/>
-</signal>
-<signal name="PC1">
-<contactref element="U1" pad="24"/>
-<wire x1="17.2974" y1="32.76" x2="16.008" y2="32.76" width="0.254" layer="1"/>
-<wire x1="16.008" y1="32.76" x2="15.748" y2="33.02" width="0.254" layer="1"/>
-<via x="15.748" y="33.02" extent="1-16" drill="0.3302" shape="octagon"/>
-<wire x1="15.748" y1="33.02" x2="14.9098" y2="33.8582" width="0.254" layer="16"/>
-<wire x1="14.9098" y1="33.8582" x2="12.2682" y2="33.8582" width="0.254" layer="16"/>
-<contactref element="AT_PINS" pad="7"/>
-<wire x1="12.2682" y1="33.8582" x2="12.2174" y2="33.8582" width="0.2032" layer="16"/>
-<wire x1="12.2174" y1="33.8582" x2="10.9728" y2="32.6136" width="0.254" layer="16"/>
 </signal>
 <signal name="BT_VOL_UP">
@@
 <via x="62.23" y="40.2082" extent="1-16" drill="0.6" shape="octagon"/>
 <wire x1="62.23" y1="40.2082" x2="62.23" y2="48.26" width="0.4064" layer="16"/>
+<contactref element="U1" pad="24"/>
+<wire x1="16.008" y1="32.76" x2="15.748" y2="33.02" width="0.254" layer="1"/>
+<via x="15.748" y="33.02" extent="1-16" drill="0.3302" shape="octagon"/>
+<wire x1="15.748" y1="33.02" x2="14.9098" y2="33.8582" width="0.254" layer="16"/>
+<wire x1="14.9098" y1="33.8582" x2="12.2682" y2="33.8582" width="0.254" layer="16"/>
+<contactref element="AT_PINS" pad="7"/>
+<wire x1="12.2682" y1="33.8582" x2="12.2174" y2="33.8582" width="0.2032" layer="16"/>
+<wire x1="12.2174" y1="33.8582" x2="10.9728" y2="32.6136" width="0.254" layer="16"/>
+<wire x1="16.008" y1="32.76" x2="17.2974" y2="32.76" width="0.254" layer="1"/>
+<wire x1="17.2974" y1="32.76" x2="60.1472" y2="40.132" width="0" layer="19" extent="1-1"/>
 </signal>
 <signal name="CHG_PG">
